Commit message: renamed pioneer model and added two 3d nerve stages

File: resources/models/pioneer/defs/pioneer.xacro (robot description, xacro)
@@ -4,5 +4,5 @@
      https://github.com/allenh1/p2os
      Note that the pioneers in p2os have no sensors. -->
-<robot name="pioneer3dx" xmlns:xacro="http://ros.org/wiki/xacro">
-  <xacro:include filename="$(find uml_3d_race)/resources/models/pioneer3dx/defs/pioneer3dx_body.xacro"/>
+<robot name="pioneer" xmlns:xacro="http://ros.org/wiki/xacro">
+  <xacro:include filename="$(find uml_3d_race)/resources/models/pioneer/defs/pioneer_body.xacro"/>
 </robot>

File: resources/models/pioneer/defs/pioneer_body.xacro (robot description, xacro)
@@ -3,5 +3,5 @@
   <!-- CONFIGURATION SETUP - - - - - - - - - - - - - - - - - - - - - - - - - -->
   <!-- Load configuration settings for a frontal laser -->
-  <xacro:property name="front_yaml_file" value="$(find uml_3d_race)/resources/models/pioneer3dx/config/frontlaser_config.yaml" />
+  <xacro:property name="front_yaml_file" value="$(find uml_3d_race)/resources/models/pioneer/config/frontlaser_config.yaml" />
   <!-- Read all the yaml properties into a list named front_config -->
   <xacro:property name="front_config" value="${load_yaml(front_yaml_file)}"/>
@@ -9,5 +9,5 @@
   <xacro:property name="front_laser" value="${front_config['enabled']}" />
   <!-- Load configuration settings for a rear laser -->
-  <xacro:property name="rear_yaml_file" value="$(find uml_3d_race)/resources/models/pioneer3dx/config/rearlaser_config.yaml" />
+  <xacro:property name="rear_yaml_file" value="$(find uml_3d_race)/resources/models/pioneer/config/rearlaser_config.yaml" />
   <!-- Read all the yaml properties into a list named rear_config -->
   <xacro:property name="rear_config" value="${load_yaml(rear_yaml_file)}"/>
@@ -15,5 +15,5 @@
   <xacro:property name="rear_laser" value="${rear_config['enabled']}" />
   <!-- Load configuration settings for a kinect -->
-  <xacro:property name="kinect_yaml_file" value="$(find uml_3d_race)/resources/models/pioneer3dx/config/kinect_config.yaml" />
+  <xacro:property name="kinect_yaml_file" value="$(find uml_3d_race)/resources/models/pioneer/config/kinect_config.yaml" />
   <!-- Read all the yaml properties into a list named rear_config -->
   <xacro:property name="kinect_config" value="${load_yaml(kinect_yaml_file)}"/>
@@ -22,9 +22,9 @@
   <!-- LOAD MACROS - - - - - - - - - - - - - - - - - - - - - - - - - - - - - -->
   <!-- Creates a macro for creating the wheel links (called towards the end of the file) -->
-  <xacro:include filename="$(find uml_3d_race)/resources/models/pioneer3dx/defs/pioneer3dx_wheel.xacro"/>
+  <xacro:include filename="$(find uml_3d_race)/resources/models/pioneer/defs/pioneer_wheel.xacro"/>
   <!-- Creates a macro for adding laser sensors (called towards the end of the file) -->
-  <xacro:include filename="$(find uml_3d_race)/resources/models/pioneer3dx/defs/pioneer3dx_lasers.xacro"/>
+  <xacro:include filename="$(find uml_3d_race)/resources/models/pioneer/defs/pioneer_lasers.xacro"/>
   <!-- Creates a macro for adding a kinect sensor (called towards the end of the file) -->
-  <xacro:include filename="$(find uml_3d_race)/resources/models/pioneer3dx/defs/pioneer3dx_kinect.xacro"/>
+  <xacro:include filename="$(find uml_3d_race)/resources/models/pioneer/defs/pioneer_kinect.xacro"/>
   <!-- ROBOT DESCRIPTION - - - - - - - - - - - - - - - - - - - - - - - - - - -->
   <!-- Chassis description -->

File: resources/models/pioneer/defs/pioneer_wheel.xacro (robot description, xacro)
@@ -17,5 +17,5 @@
         <geometry name="pioneer_geom">
           <mesh filename="file://$(arg model_dir)/${suffix}_wheel.stl"/>
-          <!-- <mesh filename="package://resources/models/pioneer3dx/meshes/${suffix}_wheel.stl"/> -->
+          <!-- <mesh filename="package://resources/models/pioneer/meshes/${suffix}_wheel.stl"/> -->
         </geometry>
         <material name="WheelBlack">
