Commit message: added collision detection and a test node that prints the collision coordinates

File: resources/models/pioneer/defs/pioneer_body.xacro (robot description, xacro)
@@ -1,315 +1,297 @@
 <?xml version="1.0"?>
 <robot xmlns:xacro="http://ros.org/wiki/xacro">
-  <!-- CONFIGURATION SETUP - - - - - - - - - - - - - - - - - - - - - - - - - -->
-  <!-- Load configuration settings for a frontal laser -->
-  <xacro:property name="front_yaml_file" value="$(find uml_3d_race)/resources/models/pioneer/config/frontlaser_config.yaml" />
-  <!-- Read all the yaml properties into a list named front_config -->
-  <xacro:property name="front_config" value="${load_yaml(front_yaml_file)}"/>
-  <!-- An example of how to access properties within the list -->
-  <xacro:property name="front_laser" value="${front_config['enabled']}" />
-  <!-- Load configuration settings for a rear laser -->
-  <xacro:property name="rear_yaml_file" value="$(find uml_3d_race)/resources/models/pioneer/config/rearlaser_config.yaml" />
-  <!-- Read all the yaml properties into a list named rear_config -->
-  <xacro:property name="rear_config" value="${load_yaml(rear_yaml_file)}"/>
-  <!-- An example of how to access properties within the list -->
-  <xacro:property name="rear_laser" value="${rear_config['enabled']}" />
-  <!-- Load configuration settings for a kinect -->
-  <xacro:property name="kinect_yaml_file" value="$(find uml_3d_race)/resources/models/pioneer/config/kinect_config.yaml" />
-  <!-- Read all the yaml properties into a list named rear_config -->
-  <xacro:property name="kinect_config" value="${load_yaml(kinect_yaml_file)}"/>
-  <!-- An example of how to access properties within the list -->
-  <xacro:property name="kinect" value="${kinect_config['enabled']}" />
-  <!-- LOAD MACROS - - - - - - - - - - - - - - - - - - - - - - - - - - - - - -->
-  <!-- Creates a macro for creating the wheel links (called towards the end of the file) -->
-  <xacro:include filename="$(find uml_3d_race)/resources/models/pioneer/defs/pioneer_wheel.xacro"/>
-  <!-- Creates a macro for adding laser sensors (called towards the end of the file) -->
-  <xacro:include filename="$(find uml_3d_race)/resources/models/pioneer/defs/pioneer_lasers.xacro"/>
-  <!-- Creates a macro for adding a kinect sensor (called towards the end of the file) -->
-  <xacro:include filename="$(find uml_3d_race)/resources/models/pioneer/defs/pioneer_kinect.xacro"/>
-  <!-- ROBOT DESCRIPTION - - - - - - - - - - - - - - - - - - - - - - - - - - -->
-  <!-- Chassis description -->
-  <link name="base_link">
-    <!-- Inertial base_link property moved to weight_link below -->
-  	<!-- CHECK THESE VALUES. THEY MAY BE WRONG. -->
-  	<!-- <inertial>
+	<!-- CONFIGURATION SETUP - - - - - - - - - - - - - - - - - - - - - - - - - -->
+	<!-- Load configuration settings for a frontal laser -->
+	<xacro:property name="front_yaml_file" value="$(find uml_3d_race)/resources/models/pioneer/config/frontlaser_config.yaml" />
+	<!-- Read all the yaml properties into a list named front_config -->
+	<xacro:property name="front_config" value="${load_yaml(front_yaml_file)}"/>
+	<!-- An example of how to access properties within the list -->
+	<xacro:property name="front_laser" value="${front_config['enabled']}" />
+	<!-- Load configuration settings for a rear laser -->
+	<xacro:property name="rear_yaml_file" value="$(find uml_3d_race)/resources/models/pioneer/config/rearlaser_config.yaml" />
+	<!-- Read all the yaml properties into a list named rear_config -->
+	<xacro:property name="rear_config" value="${load_yaml(rear_yaml_file)}"/>
+	<!-- An example of how to access properties within the list -->
+	<xacro:property name="rear_laser" value="${rear_config['enabled']}" />
+	<!-- Load configuration settings for a kinect -->
+	<xacro:property name="kinect_yaml_file" value="$(find uml_3d_race)/resources/models/pioneer/config/kinect_config.yaml" />
+	<!-- Read all the yaml properties into a list named rear_config -->
+	<xacro:property name="kinect_config" value="${load_yaml(kinect_yaml_file)}"/>
+	<!-- An example of how to access properties within the list -->
+	<xacro:property name="kinect" value="${kinect_config['enabled']}" />
+	<!-- LOAD MACROS - - - - - - - - - - - - - - - - - - - - - - - - - - - - - -->
+	<!-- Creates a macro for creating the wheel links (called towards the end of the file) -->
+	<xacro:include filename="$(find uml_3d_race)/resources/models/pioneer/defs/pioneer_wheel.xacro"/>
+	<!-- Creates a macro for adding laser sensors (called towards the end of the file) -->
+	<xacro:include filename="$(find uml_3d_race)/resources/models/pioneer/defs/pioneer_lasers.xacro"/>
+	<!-- Creates a macro for adding a kinect sensor (called towards the end of the file) -->
+	<xacro:include filename="$(find uml_3d_race)/resources/models/pioneer/defs/pioneer_kinect.xacro"/>
+	<!-- ROBOT DESCRIPTION - - - - - - - - - - - - - - - - - - - - - - - - - - -->
+	<!-- Chassis description -->
+	<link name="base_link">
+		<!-- Inertial base_link property moved to weight_link below -->
+		<!-- CHECK THESE VALUES. THEY MAY BE WRONG. -->
+		<!-- <inertial>
   	  <mass value="20.0"/>
   	  <origin xyz="-0.045 0 0.148"/>
-  	  <inertia ixx="0.3338" ixy="0.0" ixz="0.0"
-  			       iyy="0.4783" iyz="0.0" izz="0.3338"/>
+  	  <inertia ixx="0.3338" ixy="0.0" ixz="0.0" iyy="0.4783" iyz="0.0" izz="0.3338"/>
   	</inertial> -->
-  	<visual>
-  	  <origin xyz="-0.045 0 0.148" rpy="0 0 0"/>
-  	  <geometry name="pioneer_geom">
-    		<mesh filename="file://$(arg model_dir)/chassis.stl"/>
-  	  </geometry>
-  	  <material name="ChassisRed">
-    		<color rgba="0.851 0.0 0.0 1.0"/>
-  	  </material>
-  	</visual>
-  	<collision>
-  	  <origin xyz="-0.045 0 0.148" rpy="0 0 0"/>
-  	  <geometry>
-        <box size="0.42 0.28 0.17"/>
-  	  </geometry>
-  	</collision>
-  </link>
-  <gazebo reference="base_link">
-  	<material value="Gazebo/Red"/>
-  </gazebo>
-  <!-- In verbose mode, gazebo complains that KDL does not support a base_link with interia
+		<visual>
+			<origin xyz="-0.045 0 0.148" rpy="0 0 0"/>
+			<geometry name="pioneer_geom">
+				<mesh filename="file://$(arg model_dir)/chassis.stl"/>
+			</geometry>
+			<material name="ChassisRed">
+				<color rgba="0.851 0.0 0.0 1.0"/>
+			</material>
+		</visual>
+		<collision name="robot_collision">
+			<origin xyz="-0.045 0 0.148" rpy="0 0 0"/>
+			<geometry>
+				<box size="0.42 0.28 0.17"/>
+			</geometry>
+		</collision>
+	</link>
+	<gazebo reference="base_link">
+		<material value="Gazebo/Red"/>
+		<!-- Adds collision detection-->
+		<sensor type="contact" name="robot_contact_sensor">
+			<update_rate>100.0</update_rate>
+			<always_on>1</always_on>
+			<contact>
+				<collision>base_link_fixed_joint_lump__robot_collision_collision</collision>
+			</contact>
+			<plugin name="robot_bumper_controller" filename="libgazebo_ros_bumper.so">
+				<alwaysOn>true</alwaysOn>
+				<updateRate>100.0</updateRate>
+				<bumperTopicName>/pioneer/bumper_contact</bumperTopicName>
+				<frameName>base_link</frameName>
+			</plugin>
+		</sensor>
+	</gazebo>
+	<!-- In verbose mode, gazebo complains that KDL does not support a base_link with interia
        so this is a dummy link with the intertial attached to base_link -->
-  <link name="weight_link">
-    <!-- CHECK THESE VALUES. THEY MAY BE WRONG. -->
-    <inertial>
-      <mass value="20.0"/>
-      <origin xyz="-0.045 0 0.148"/>
-      <inertia ixx="0.3338" ixy="0.0" ixz="0.0"
-               iyy="0.4783" iyz="0.0" izz="0.3338"/>
-    </inertial>
-  </link>
-  <joint name="weight_joint" type="fixed">
-    <origin xyz="-0.04 0 -0.02" rpy="0 0 0"/>
-    <parent link="base_link"/>
-    <child link="weight_link"/>
-  </joint>
-  <link name="top_plate">
-  	<inertial>
-  	  <mass value="0.01"/>
-  	  <origin xyz="0 0 0"/>
-  	  <inertia ixx="1" ixy="0" ixz="0"
-  			       iyy="1" iyz="0" izz="1"/>
-  	</inertial>
-  	<visual>
-  	  <origin xyz="0 0 0" rpy="0 0 0"/>
-  	  <geometry name="pioneer_geom">
-    		<mesh filename="file://$(arg model_dir)/top.stl"/>
-  	  </geometry>
-  	  <material name="TopBlack">
-    		<color rgba="0.038 0.038 0.038 1.0"/>
-  	  </material>
-  	</visual>
-  </link>
-  <gazebo reference="top_plate">
-  	<material value="Gazebo/Black"/>
-  </gazebo>
-  <joint name="base_top_joint" type="fixed">
-  	<origin xyz="-0.045 0 0.24" rpy="0 0 0"/>
-  	<parent link="base_link"/>
-  	<child link="top_plate"/>
-  </joint>
-  <!-- Swivel -->
-  <link name="swivel_link">
-  	<inertial>
-  	  <mass value="0.1"/>
-  	  <origin xyz="0 0 0"/>
-  	  <inertia ixx="0.01" ixy="0" ixz="0"
-  			       iyy="0.01" iyz="0" izz="0.01"/>
-  	</inertial>
-  	<visual>
-  	  <origin xyz="0 0 0" rpy="0 0 0"/>
-  	  <geometry name="pioneer_geom">
-    		<mesh filename="file://$(arg model_dir)/swivel.stl"/>
-  	  </geometry>
-  	  <material name="swivel">
-    		<color rgba="0.5 0.5 0.5 1"/>
-  	  </material>
-  	</visual>
-  </link>
-  <gazebo reference="swivel_link">
-  	<material value="Gazebo/Black"/>
-  </gazebo>
-  <joint name="base_swivel_joint" type="continuous">
-  	<origin xyz="-0.185 0 0.055" rpy="0 0 0"/>
-  	<parent link="base_link"/>
-  	<child link="swivel_link"/>
-  	<axis xyz="0 0 1"/>
-    <limit effort="100" velocity="100" k_velocity="0" />
-    <joint_properties damping="0.0" friction="0.0" />
-  </joint>
-  <!-- Center Wheel + Hubcap -->
-  <link name="center_hubcap">
-    <inertial>
-  	  <mass value="0.01"/>
-  	  <origin xyz="0 0 0"/>
-  	  <inertia ixx="0.012411765597" ixy="-0.000711733678" ixz="0.00050272983"
-  			       iyy="0.015218160428" iyz="-0.000004273467" izz="0.011763977943"/>
-  	</inertial>
-  	<visual>
-  	  <origin xyz="0 0 0" rpy="0 0 0"/>
-  	  <geometry name="pioneer_geom">
-    		<mesh filename="file://$(arg model_dir)/center_hubcap.stl"/>
-  	  </geometry>
-  	  <material name="swivel">
-    		<color rgba="0.5 0.5 0.5 1"/>
-  	  </material>
-  	</visual>
-  </link>
-  <gazebo reference="center_hubcap">
-  	<material value="Gazebo/Black"/>
-  </gazebo>
-  <joint name="swivel_hubcap_joint" type="continuous">
-  	<origin xyz="-0.026 0 -0.016" rpy="0 0 0"/>
-  	<parent link="swivel_link"/>
-  	<child link="center_wheel"/>
-  	<axis xyz="0 1 0"/>
-  	<anchor xyz="0 0 0"/>
-    <limit effort="100" velocity="100" k_velocity="0" />
-    <joint_properties damping="0.0" friction="0.0" />
-  </joint>
-  <link name="center_wheel">
-  	<inertial>
-  	  <mass value="0.1"/>
-  	  <origin xyz="0 0 0"/>
-  	  <inertia ixx="0.012411765597" ixy="-0.000711733678" ixz="0.00050272983"
-  			       iyy="0.015218160428" iyz="-0.000004273467" izz="0.011763977943"/>
-  	</inertial>
-  	<visual>
-  	  <origin xyz="0 0 0" rpy="0 0 0"/>
-  	  <geometry name="pioneer_geom">
-    		<mesh filename="file://$(arg model_dir)/center_wheel.stl"/>
-  	  </geometry>
-  	  <material name="WheelBlack">
-    		<color rgba="0.117 0.117 0.117 1"/>
-  	  </material>
-  	</visual>
-  	<collision>
-  	  <origin xyz="0 0 0" rpy="${-3.1415927/2.0} 0 0"/>
-  	  <geometry>
-    		<cylinder radius="0.0375" length="0.0314"/>
-  	  </geometry>
-  	</collision>
-  </link>
-  <gazebo reference="center_wheel">
-  	<material value="Gazebo/Black"/>
-  </gazebo>
-  <joint name="center_wheel_joint" type="fixed">
-  	<origin xyz="-0.0035 0 -0.001" rpy="0 0 0"/>
-  	<parent link="center_wheel"/>
-  	<child link="center_hubcap"/>
-  </joint>
-  <xacro:p3dx_wheel suffix="left" parent="base_link" reflect="1"/>
-  <xacro:p3dx_wheel suffix="right" parent="base_link" reflect="-1"/>
-  <!-- Front + Back Sonar -->
-  <link name="front_sonar">
-  	<inertial>
-  	  <mass value="0.0001"/>
-  	  <origin xyz="0 0 0"/>
-  	  <inertia ixx="1" ixy="0" ixz="0"
-  			       iyy="1" iyz="0" izz="1"/>
-  	</inertial>
-  	<visual>
-  	  <origin xyz="0 0 0" rpy="0 0 0"/>
-  	  <geometry name="pioneer_geom">
-    		<mesh filename="file://$(arg model_dir)/front_sonar.stl"/>
-  	  </geometry>
-  	  <material name="SonarYellow">
-    		<color rgba="0.715 0.583 0.210 1.0"/>
-  	  </material>
-  	</visual>
-  </link>
-  <gazebo reference="front_sonar">
-  	<material value="Gazebo/Yellow"/>
-  </gazebo>
-  <joint name="base_front_joint" type="fixed">
-  	<origin xyz="-0.198 0 0.208" rpy="0 0 0"/>
-  	<parent link="base_link"/>
-  	<child link="front_sonar"/>
-  </joint>
-  <link name="back_sonar">
-  	<inertial>
-  	  <mass value="0.0001"/>
-  	  <origin xyz="0 0 0"/>
-  	  <inertia ixx="1" ixy="0" ixz="0"
-  			       iyy="1" iyz="0" izz="1"/>
-  	</inertial>
-  	<visual>
-  	  <origin xyz="0 0 0" rpy="0 0 0"/>
-  	  <geometry name="pioneer_geom">
-    		<mesh filename="file://$(arg model_dir)/back_sonar.stl"/>
-  	  </geometry>
-  	  <material name="SonarYellow">
-    		<color rgba="0.715 0.583 0.210 1.0"/>
-  	  </material>
-  	</visual>
-  </link>
-  <gazebo reference="back_sonar">
-	   <material value="Gazebo/Yellow"/>
-  </gazebo>
-  <joint name="base_back_joint" type="fixed">
-  	<origin xyz="0.109 0 0.209" rpy="0 0 0"/>
-  	<parent link="base_link"/>
-  	<child link="back_sonar"/>
-  </joint>
-  <gazebo>
-    <!-- Robot locomotion plugin -->
-  	<plugin name="differential_drive_controller" filename="libgazebo_ros_diff_drive.so">
-      <legacyMode>false</legacyMode>
-      <alwaysOn>true</alwaysOn>
-  	  <updateRate>100.0</updateRate>
-  	  <leftJoint>base_left_wheel_joint</leftJoint>
-      <rightJoint>base_right_wheel_joint</rightJoint>
-  	  <wheelSeparation>0.32</wheelSeparation>
-  	  <wheelDiameter>0.18</wheelDiameter>
-  	  <wheelTorque>5</wheelTorque>
-      <wheelAcceleration>0</wheelAcceleration>
-      <robotNamespace>$(arg model_name)</robotNamespace>
-  	  <commandTopic>cmd_vel</commandTopic>
-  	  <odometryTopic>odom</odometryTopic>
-  	  <odometryFrame>odom</odometryFrame>
-      <robotBaseFrame>base_link</robotBaseFrame>
-      <publishTf>1</publishTf>
-      <publishWheelTF>true</publishWheelTF>
-      <publishOdomTF>true</publishOdomTF>
-      <publishWheelJointState>true</publishWheelJointState>
-      <rosDebugLevel>Warn</rosDebugLevel>
-  	</plugin>
-    <!-- Fake localization plugin -->
-    <plugin name="ground_truth_odometry" filename="libgazebo_ros_p3d.so">
-  	  <alwaysOn>true</alwaysOn>
-  	  <updateRate>100.0</updateRate>
-  	  <bodyName>base_link</bodyName>
-  	  <topicName>base_pose_ground_truth</topicName>
-  	  <gaussianNoise>0.01</gaussianNoise>
-  	  <frameName>map</frameName>-->
-      <!-- initialize odometry for fake localization-->
-  	  <xyzOffsets>0 0 0</xyzOffsets>
-  	  <rpyOffsets>0 0 0</rpyOffsets>
-  	</plugin>
-  </gazebo>
-  <!-- If enabled is set to true, add the front laser. -->
-  <xacro:if value="${front_laser == 1}">
-    <xacro:add_laser descriptor="${front_config['descriptor']}"
-                     visualize="${front_config['visualize']}"
-                     x="${front_config['x']}"
-                     y="${front_config['y']}"
-                     z="${front_config['z']}"
-                     yaw="${front_config['yaw']}"
-                     min="${front_config['min_angle']}"
-                     max="${front_config['max_angle']}"
-                     samples="${front_config['ray_count']}"
-                     range="${front_config['range']}"/>
-  </xacro:if>
-  <!-- If enabled is set to true, add the rear laser. -->
-  <xacro:if value="${rear_laser == 1}">
-    <xacro:add_laser descriptor="${rear_config['descriptor']}"
-                     visualize="${rear_config['visualize']}"
-                     x="${rear_config['x']}"
-                     y="${rear_config['y']}"
-                     z="${rear_config['z']}"
-                     yaw="${rear_config['yaw']}"
-                     min="${rear_config['min_angle']}"
-                     max="${rear_config['max_angle']}"
-                     samples="${rear_config['ray_count']}"
-                     range="${rear_config['range']}"/>
-  </xacro:if>
-  <!-- If enabled is set to true, add the kinect. -->
-  <xacro:if value="${kinect == 1}">
-    <xacro:add_kinect descriptor="${kinect_config['descriptor']}"
-                      x="${kinect_config['x']}"
-                      y="${kinect_config['y']}"
-                      height="${kinect_config['height']}"
-                      pan="${kinect_config['pan']}"
-                      tilt="${kinect_config['tilt']}"
-                      far_clip="${kinect_config['far_clip']}"/>
-  </xacro:if>
+	<link name="weight_link">
+		<!-- CHECK THESE VALUES. THEY MAY BE WRONG. -->
+		<inertial>
+			<mass value="20.0"/>
+			<origin xyz="-0.045 0 0.148"/>
+			<inertia ixx="0.3338" ixy="0.0" ixz="0.0" iyy="0.4783" iyz="0.0" izz="0.3338"/>
+		</inertial>
+	</link>
+	<joint name="weight_joint" type="fixed">
+		<origin xyz="-0.04 0 -0.02" rpy="0 0 0"/>
+		<parent link="base_link"/>
+		<child link="weight_link"/>
+	</joint>
+	<link name="top_plate">
+		<inertial>
+			<mass value="0.01"/>
+			<origin xyz="0 0 0"/>
+			<inertia ixx="1" ixy="0" ixz="0" iyy="1" iyz="0" izz="1"/>
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
Commit message: changed collision hitbox

File: resources/models/pioneer/defs/pioneer_body.xacro (robot description, xacro)
@@ -49,5 +49,5 @@
 			<origin xyz="-0.045 0 0.148" rpy="0 0 0"/>
 			<geometry>
-				<box size="0.42 0.28 0.17"/>
+				<mesh filename="file://$(arg model_dir)/collision.stl"/>
 			</geometry>
 		</collision>

Commit message: improved run_test script by merging the log_data script to avoid annoying process management

File: resources/models/pioneer/defs/pioneer_body.xacro (robot description, xacro)
@@ -3,5 +3,5 @@
 	<!-- CONFIGURATION SETUP - - - - - - - - - - - - - - - - - - - - - - - - - -->
 	<!-- Load configuration settings for a frontal laser -->
-	<xacro:property name="front_yaml_file" value="$(find uml_3d_race)/resources/models/pioneer/config/frontlaser_config.yaml" />
+	<xacro:property name="front_yaml_file" value="$(find uml_3d_race)/resources/config/pioneer/frontlaser_config.yaml" />
 	<!-- Read all the yaml properties into a list named front_config -->
 	<xacro:property name="front_config" value="${load_yaml(front_yaml_file)}"/>
@@ -9,5 +9,5 @@
 	<xacro:property name="front_laser" value="${front_config['enabled']}" />
 	<!-- Load configuration settings for a rear laser -->
-	<xacro:property name="rear_yaml_file" value="$(find uml_3d_race)/resources/models/pioneer/config/rearlaser_config.yaml" />
+	<xacro:property name="rear_yaml_file" value="$(find uml_3d_race)/resources/config/pioneer/rearlaser_config.yaml" />
 	<!-- Read all the yaml properties into a list named rear_config -->
 	<xacro:property name="rear_config" value="${load_yaml(rear_yaml_file)}"/>
@@ -15,5 +15,5 @@
 	<xacro:property name="rear_laser" value="${rear_config['enabled']}" />
 	<!-- Load configuration settings for a kinect -->
-	<xacro:property name="kinect_yaml_file" value="$(find uml_3d_race)/resources/models/pioneer/config/kinect_config.yaml" />
+	<xacro:property name="kinect_yaml_file" value="$(find uml_3d_race)/resources/config/pioneer/kinect_config.yaml" />
 	<!-- Read all the yaml properties into a list named rear_config -->
 	<xacro:property name="kinect_config" value="${load_yaml(kinect_yaml_file)}"/>
