Commit message: worked on fetch and added launch file for obstacle bot

File: resources/models/obstacle_bot/obstacle_bot.xacro (robot description, xacro)
@@ -4,6 +4,6 @@
   <xacro:property name="robot_radius" value="0.25" />
   <xacro:property name="antenna_len" value="0.2" />
-  <xacro:property name="robot_height" value="$(arg height)" />
-  <xacro:property name="robot_radius" value="$(arg radius)" />
+  <!-- <xacro:property name="robot_height" value="$(arg height)" />
+  <xacro:property name="robot_radius" value="$(arg radius)" /> -->
   <!-- root link, on the ground just below the model origin -->
   <link name="base_footprint">
